File: Hardware/SparkFun_Thermocouple_Breakout.brd (EAGLE design)
At the start: 30 x 19.8 mm, 17 parts, among them U1 MAX31855K

Commit message: Added testpoints for the thermocouple connections
Parts:
- added TP1, TP2: TEST-POINTTP_15TH_THRU, SparkFun-Passives:TP_15TH
Connections:
- net N$4: now also TP1.P$1
- net N$5: now also TP2.P$1
Routing:
- net N$4: track 3.02 -> 5.22 mm
- net N$5: track 3.02 -> 4.04 mm
Changed lines of the file:
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@@
 <setting verticaltext="up"/>
 </settings>
-<grid distance="0.005" unitdist="inch" unit="inch" style="lines" multiple="1" display="yes" altdistance="0.005" altunitdist="inch" altunit="inch"/>
+<grid distance="0.01" unitdist="inch" unit="inch" style="lines" multiple="1" display="yes" altdistance="0.005" altunitdist="inch" altunit="inch"/>
 <layers>
 <layer number="1" name="Top" color="4" fill="1" visible="yes" active="yes"/>
@@
 <element name="LOGO3" library="SparkFun-Aesthetics" package="SFE_LOGO_NAME_FLAME_.1" value="SFE_LOGO_NAME_FLAME.1_INCH" x="28.194" y="15.367" rot="MR270"/>
 <element name="LOGO4" library="SparkFun-Aesthetics" package="OSHW-LOGO-S" value="OSHW-LOGOS" x="14.859" y="9.906" rot="MR270"/>
+<element name="TP1" library="SparkFun-Passives" package="TP_15TH" value="TEST-POINTTP_15TH_THRU" x="16.256" y="15.24"/>
+<element name="TP2" library="SparkFun-Passives" package="TP_15TH" value="TEST-POINTTP_15TH_THRU" x="16.256" y="4.572"/>
 </elements>
 <signals>
@@
 <contactref element="L1" pad="2"/>
 <contactref element="JP2" pad="-"/>
-<wire x1="15.24" y1="5.754" x2="15.24" y2="3.81" width="0.4064" layer="1"/>
+<wire x1="15.24" y1="5.754" x2="15.24" y2="4.572" width="0.4064" layer="1"/>
+<wire x1="15.24" y1="4.572" x2="15.24" y2="3.81" width="0.4064" layer="1"/>
 <wire x1="15.24" y1="3.81" x2="14.478" y2="3.048" width="0.4064" layer="1"/>
+<contactref element="TP2" pad="P$1"/>
+<wire x1="16.256" y1="4.572" x2="15.24" y2="4.572" width="0.4064" layer="1"/>
 </signal>
 <signal name="N$4">
@@
 <wire x1="15.24" y1="14.058" x2="15.24" y2="16.002" width="0.4064" layer="1"/>
 <wire x1="15.24" y1="16.002" x2="14.478" y2="16.764" width="0.4064" layer="1"/>
+<contactref element="TP1" pad="P$1"/>
+<wire x1="15.24" y1="14.058" x2="15.24" y2="15.24" width="0.4064" layer="1"/>
+<wire x1="15.24" y1="15.24" x2="16.256" y2="15.24" width="0.4064" layer="1"/>
 </signal>
 </signals>
