File: Hardware/SparkFun_Thermocouple_Breakout.brd (EAGLE design)
At the start: 30 x 19.8 mm, 19 parts, among them U1 MAX31855K

Commit message: Swapped a pin
Connections:
- net N$2: now also JP1.4; no longer JP1.5
Routing:
- net N$2: track 7.63 -> 6.28 mm
Other:
- board text added: "SO"
- board text removed: "(MI)SO"
Changed lines of the file:
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@@
 <text x="2.794" y="13.716" size="1.016" layer="21" font="vector" ratio="15" align="center-left">VCC</text>
 <text x="2.794" y="3.556" size="1.016" layer="21" font="vector" ratio="15" align="center-left">!CS</text>
-<text x="2.794" y="6.096" size="1.016" layer="21" font="vector" ratio="15" align="center-left">(MI)SO</text>
-<text x="2.794" y="8.636" size="1.016" layer="21" font="vector" ratio="15" align="center-left">NC</text>
+<text x="2.794" y="8.636" size="1.016" layer="21" font="vector" ratio="15" align="center-left">SO</text>
+<text x="2.794" y="6.096" size="1.016" layer="21" font="vector" ratio="15" align="center-left">NC</text>
 <text x="2.794" y="11.176" size="1.016" layer="21" font="vector" ratio="15" align="center-left">SCK</text>
 <text x="2.794" y="16.256" size="1.016" layer="21" font="vector" ratio="15" align="center-left">GND</text>
@@
 <rectangle x1="12.7" y1="8.382" x2="13.208" y2="8.89" layer="41"/>
 <text x="2.794" y="3.556" size="1.016" layer="22" font="vector" ratio="15" rot="MR0" align="center-right">!CS</text>
-<text x="2.794" y="6.096" size="1.016" layer="22" font="vector" ratio="15" rot="MR0" align="center-right">(MI)SO</text>
-<text x="2.794" y="8.636" size="1.016" layer="22" font="vector" ratio="15" rot="MR0" align="center-right">NC</text>
+<text x="2.794" y="8.636" size="1.016" layer="22" font="vector" ratio="15" rot="MR0" align="center-right">SO</text>
+<text x="2.794" y="6.096" size="1.016" layer="22" font="vector" ratio="15" rot="MR0" align="center-right">NC</text>
 <text x="2.794" y="11.176" size="1.016" layer="22" font="vector" ratio="15" rot="MR0" align="center-right">SCK</text>
 <text x="2.794" y="16.256" size="1.016" layer="22" font="vector" ratio="15" rot="MR0" align="center-right">GND</text>
@@
 <signal name="N$2">
 <contactref element="U1" pad="7"/>
-<contactref element="JP1" pad="5"/>
-<wire x1="2.286" y1="7.112" x2="1.27" y2="6.096" width="0.4064" layer="1"/>
-<wire x1="5.207" y1="8.255" x2="4.064" y2="7.112" width="0.4064" layer="1"/>
-<wire x1="4.064" y1="7.112" x2="2.286" y2="7.112" width="0.4064" layer="1"/>
-<wire x1="5.207" y1="8.255" x2="5.207" y2="8.763" width="0.4064" layer="1"/>
-<wire x1="5.207" y1="8.763" x2="5.715" y2="9.271" width="0.4064" layer="1"/>
-<wire x1="5.715" y1="9.271" x2="7.2898" y2="9.271" width="0.4064" layer="1"/>
+<contactref element="JP1" pad="4"/>
+<wire x1="7.2898" y1="9.271" x2="1.905" y2="9.271" width="0.4064" layer="1"/>
+<wire x1="1.905" y1="9.271" x2="1.27" y2="8.636" width="0.4064" layer="1"/>
 </signal>
 <signal name="N$8">
